File: nTerm2-S FT231.kicad_sch (KiCad schematic)
At the start: 122 parts, among them J1 VGA, J2 Keyboard, J3 Mouse, J4 Line-out/Speaker, J5 RS-232 V.24, J6 USB_C_Receptacle_USB2.0_16P, J7 Line-out/Speaker, K1 IM41 3V, K2 IM41 3V, K3 IM41 3V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

Commit message: And here's revision 0.08. I added some solder bridges so that people can choose to place the relays and driver circuits, or forego on the switching option and just be happy with RxD, TxD, RTS and CTS hardwired on the RS-232 port. It was always possible to bypass using a patch wire or course, but this is just a little more friendly.
Parts:
- added OPT2, OPT3, OPT4, OPT5: Bypass, Library:SolderJumper-3_P1.3mm_Open_RoundedPad1.0x1.5mm_NumberLabels, symbol nTerm2-S:SolderJumper_3_Open
- renumbered JP1 to OPT1
Connections:
- net CTS: now also OPT5.2 (C); no longer K2.6
- net RTS: now also OPT4.2 (C); no longer K2.3
- net RxD: now also OPT2.2 (C); no longer K1.3
- net TxD: now also OPT3.2 (C); no longer K1.6
- net _CTS: now also OPT5.3 (B)
- net _RTS: now also OPT4.3 (B)
- net _RXD: now also OPT2.3 (B)
- net _TXD: now also OPT3.3 (B)
- new net: K1.6, OPT3.1 (A)
- new net: K1.3, OPT2.1 (A)
- new net: K2.6, OPT5.1 (A)
- new net: K2.3, OPT4.1 (A)
Other:
- note added: "OPT2...OPT5 Bypass: You can choose to place the switching relays and driver circuitry or not. * Solder bridges 1-2 and assemble all relays and their driver circuits. You will have switchable normal/null modem and DTR/DSR then. * Solder bridges 2-3 and leave out all the circuitry. You will have RxD, TxD, RTS and CTS hardwired to the RS-232 connector then. It will save you some cost if you don't ne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"
